Commit message: created core URDF

File: description/robot_core.xacro (robot description, xacro)
@@ -19,4 +19,13 @@
             <origin xyz="0.375 0.25 0.15" rpy="0 0 0" />
         </visual>
+        <collision>
+            <origin xyz="0.375 0.25 0.15"/>
+            <geometry>
+                <box size="0.75 0.5 0.3"/>
+            </geometry>
+        </collision>
+        <xacro:inertial_box mass="0.5" x="0.75" y="0.5" z="0.3">
+            <origin xyz="0.375 0.25 0.15" rpy="0 0 0"/>
+        </xacro:inertial_box>
     </link>
     <link name="lobase">
@@ -28,4 +37,13 @@
             <material name="white" />
         </visual>
+        <collision>
+            <origin xyz="0 0 0"/>
+            <geometry>
+                <box size="0.6 0.3 0.15"/>
+            </geometry>
+        </collision>
+        <xacro:inertial_box mass="0.5" x="0.6" y="0.3" z="0.15">
+            <origin xyz="0 0 0" rpy="0 0 0"/>
+        </xacro:inertial_box>
     </link>
     <link name="lidar">
@@ -37,4 +55,12 @@
             <material name="white" />
         </visual>
+        <collision>
+            <geometry>
+                <cylinder radius="0.05" length="0.03"/>
+            </geometry>
+        </collision>
+        <xacro:inertial_cylinder mass="0.1" length="0.03" radius="0.05">
+            <origin xyz="0 0 0" rpy="0 0 0"/>
+        </xacro:inertial_cylinder>
     </link>
     <link name="pipe">
@@ -46,4 +72,13 @@
             <material name="green"/>
         </visual>
+        <collision>
+            <origin xyz="0 0 0"/>
+            <geometry>
+                <box size="0.04 0.04 0.65"/>
+            </geometry>
+        </collision>
+        <xacro:inertial_box mass="0.25" x="0.04" y="0.04" z="0.65">
+            <origin xyz="0 0 0" rpy="0 0 0"/>
+        </xacro:inertial_box>
     </link>
     <link name="front_left">
@@ -55,4 +90,12 @@
          <material name="grey"/>
       </visual>
+      <collision>
+            <geometry>
+                <cylinder radius="0.15" length="0.08"/>
+            </geometry>
+        </collision>
+        <xacro:inertial_cylinder mass="0.3" length="0.08" radius="0.15">
+            <origin xyz="0 0 0" rpy="0 0 0"/>
+        </xacro:inertial_cylinder>
     </link>
     <link name="front_right">
@@ -64,4 +107,12 @@
          <material name="grey"/>
       </visual>
+      <collision>
+            <geometry>
+                <cylinder radius="0.15" length="0.08"/>
+            </geometry>
+        </collision>
+        <xacro:inertial_cylinder mass="0.3" length="0.08" radius="0.15">
+            <origin xyz="0 0 0" rpy="0 0 0"/>
+        </xacro:inertial_cylinder>
     </link>
     <link name="rear_right">
@@ -73,4 +124,12 @@
          <material name="grey"/>
       </visual>
+      <collision>
+            <geometry>
+                <cylinder radius="0.15" length="0.08"/>
+            </geometry>
+        </collision>
+        <xacro:inertial_cylinder mass="0.3" length="0.08" radius="0.15">
+            <origin xyz="0 0 0" rpy="0 0 0"/>
+        </xacro:inertial_cylinder>
     </link>
     <link name="rear_left">
@@ -82,4 +141,12 @@
          <material name="grey"/>
       </visual>
+      <collision>
+            <geometry>
+                <cylinder radius="0.15" length="0.08"/>
+            </geometry>
+        </collision>
+        <xacro:inertial_cylinder mass="0.3" length="0.08" radius="0.15">
+            <origin xyz="0 0 0" rpy="0 0 0"/>
+        </xacro:inertial_cylinder>
     </link>
     <joint name="base_joint" type="fixed">

Commit message: created core URDF

File: description/robot_core.xacro (robot description, xacro)
@@ -29,4 +29,7 @@
         </xacro:inertial_box>
     </link>
+    <gazebo reference="base_link">
+      <material>Gazebo/green</material>
+    </gazebo>
     <link name="lobase">
         <visual>
@@ -47,4 +50,7 @@
         </xacro:inertial_box>
     </link>
+    <gazebo reference="lobase">
+      <material>Gazebo/white</material>
+    </gazebo>
     <link name="lidar">
         <visual>
@@ -64,4 +70,7 @@
         </xacro:inertial_cylinder>
     </link>
+    <gazebo reference="lidar">
+      <material>Gazebo/grey</material>
+    </gazebo>
     <link name="pipe">
         <visual>
@@ -82,4 +91,7 @@
         </xacro:inertial_box>
     </link>
+    <gazebo reference="pipe">
+      <material>Gazebo/grey</material>
+    </gazebo>
     <link name="front_left">
       <visual>
@@ -99,4 +111,7 @@
         </xacro:inertial_cylinder>
     </link>
+    <gazebo reference="front_left">
+      <material>Gazebo/grey</material>
+    </gazebo>
     <link name="front_right">
       <visual>
@@ -116,4 +131,7 @@
         </xacro:inertial_cylinder>
     </link>
+    <gazebo reference="front_right">
+      <material>Gazebo/grey</material>
+    </gazebo>
     <link name="rear_right">
       <visual>
@@ -133,4 +151,7 @@
         </xacro:inertial_cylinder>
     </link>
+    <gazebo reference="rear_right">
+      <material>Gazebo/grey</material>
+    </gazebo>
     <link name="rear_left">
       <visual>
@@ -150,4 +171,7 @@
         </xacro:inertial_cylinder>
     </link>
+    <gazebo reference="rear_left">
+      <material>Gazebo/grey</material>
+    </gazebo>
     <joint name="base_joint" type="fixed">
        <parent link="base_footprint"/>

Commit message: created core URDF

File: description/robot_core.xacro (robot description, xacro)
@@ -11,4 +11,13 @@
         <color rgba="1 1 1 1" />
     </material>
+    <material name="orange">
+        <color rgba="1 0.3 0.1 1"/>
+    </material>
+    <material name="blue">
+        <color rgba="0.2 0.2 1 1"/>
+    </material>
+    <material name="black">
+        <color rgba="0 0 0 1"/>
+    </material>
     <link name="base_footprint" />
     <link name="base_link">
@@ -18,4 +27,5 @@
             </geometry>
             <origin xyz="0.375 0.25 0.15" rpy="0 0 0" />
+             <material name="green" />
         </visual>
         <collision>
@@ -30,5 +40,6 @@
     </link>
     <gazebo reference="base_link">
-      <material>Gazebo/green</material>
+      <material><Gazebo/>
+      <green></green></material>
     </gazebo>
     <link name="lobase">
@@ -51,5 +62,6 @@
     </link>
     <gazebo reference="lobase">
-      <material>Gazebo/white</material>
+      <material><Gazebo/>
+      <white></white></material>
     </gazebo>
     <link name="lidar">
@@ -59,5 +71,5 @@
             </geometry>
             <origin xyz="0 0 0" rpy="0 0 0" />
-            <material name="white" />
+            <material name="blue" />
         </visual>
         <collision>
@@ -71,5 +83,6 @@
     </link>
     <gazebo reference="lidar">
-      <material>Gazebo/grey</material>
+      <material><Gazebo/>
+      <blue></blue></material>
     </gazebo>
     <link name="pipe">
@@ -79,5 +92,5 @@
             </geometry>
             <origin xyz="0 0 0" rpy="0 0 0"/>
-            <material name="green"/>
+            <material name="orange"/>
         </visual>
         <collision>
@@ -92,5 +105,6 @@
     </link>
     <gazebo reference="pipe">
-      <material>Gazebo/grey</material>
+      <material><Gazebo/>
+      <orange></orange></material>
     </gazebo>
     <link name="front_left">
@@ -100,5 +114,5 @@
          </geometry>
          <origin xyz="0 0 0" rpy="1.57 0 0"/>
-         <material name="grey"/>
+         <material name="black"/>
       </visual>
       <collision>
@@ -112,5 +126,6 @@
     </link>
     <gazebo reference="front_left">
-      <material>Gazebo/grey</material>
+      <material><Gazebo/>
+      <black></black></material>
     </gazebo>
     <link name="front_right">
@@ -120,5 +135,5 @@
          </geometry>
          <origin xyz="0 0 0" rpy="1.57 0 0"/>
-         <material name="grey"/>
+         <material name="black"/>
       </visual>
       <collision>
@@ -132,5 +147,6 @@
     </link>
     <gazebo reference="front_right">
-      <material>Gazebo/grey</material>
+      <material><Gazebo/>
+      <black></black></material>
     </gazebo>
     <link name="rear_right">
@@ -140,5 +156,5 @@
          </geometry>
          <origin xyz="0 0 0" rpy="1.57 0 0"/>
-         <material name="grey"/>
+         <material name="black"/>
       </visual>
       <collision>
@@ -152,5 +168,6 @@
     </link>
     <gazebo reference="rear_right">
-      <material>Gazebo/grey</material>
+      <material><Gazebo/>
+      <black></black></material>
     </gazebo>
     <link name="rear_left">
@@ -160,5 +177,5 @@
          </geometry>
          <origin xyz="0 0 0" rpy="1.57 0 0"/>
-         <material name="grey"/>
+         <material name="black"/>
       </visual>
       <collision>
@@ -172,5 +189,6 @@
     </link>
     <gazebo reference="rear_left">
-      <material>Gazebo/grey</material>
+      <material><Gazebo/>
+      <black></black></material>
     </gazebo>
     <joint name="base_joint" type="fixed">

Commit message: created core URDF

File: description/robot_core.xacro (robot description, xacro)
@@ -40,6 +40,5 @@
     </link>
     <gazebo reference="base_link">
-      <material><Gazebo/>
-      <green></green></material>
+          <material>Gazebo/green</material>
     </gazebo>
     <link name="lobase">
@@ -62,6 +61,5 @@
     </link>
     <gazebo reference="lobase">
-      <material><Gazebo/>
-      <white></white></material>
+      <material>Gazebo/white</material>
     </gazebo>
     <link name="lidar">
@@ -83,6 +81,5 @@
     </link>
     <gazebo reference="lidar">
-      <material><Gazebo/>
-      <blue></blue></material>
+      <material>Gazebo/blue</material>
     </gazebo>
     <link name="pipe">
@@ -105,6 +102,5 @@
     </link>
     <gazebo reference="pipe">
-      <material><Gazebo/>
-      <orange></orange></material>
+      <material>Gazebo/orange</material>
     </gazebo>
     <link name="front_left">
@@ -126,6 +122,5 @@
     </link>
     <gazebo reference="front_left">
-      <material><Gazebo/>
-      <black></black></material>
+      <material>Gazebo/black</material>
     </gazebo>
     <link name="front_right">
@@ -147,6 +142,5 @@
     </link>
     <gazebo reference="front_right">
-      <material><Gazebo/>
-      <black></black></material>
+      <material>Gazebo/black</material>
     </gazebo>
     <link name="rear_right">
@@ -168,6 +162,5 @@
     </link>
     <gazebo reference="rear_right">
-      <material><Gazebo/>
-      <black></black></material>
+      <material>Gazebo/black</material>
     </gazebo>
     <link name="rear_left">
@@ -189,6 +182,5 @@
     </link>
     <gazebo reference="rear_left">
-      <material><Gazebo/>
-      <black></black></material>
+      <material>Gazebo/black</material>
     </gazebo>
     <joint name="base_joint" type="fixed">

Commit message: created core URDF

File: description/robot_core.xacro (robot description, xacro)
@@ -21,4 +21,5 @@
     </material>
     <link name="base_footprint" />
+    </link>
     <link name="base_link">
         <visual>

Commit message: created core URDE

File: description/robot_core.xacro (robot description, xacro)
@@ -21,5 +21,4 @@
     </material>
     <link name="base_footprint" />
-    </link>
     <link name="base_link">
         <visual>

Commit message: created core URDF

File: description/robot_core.xacro (robot description, xacro)
@@ -39,7 +39,4 @@
         </xacro:inertial_box>
     </link>
-    <gazebo reference="base_link">
-          <material>Gazebo/green</material>
-    </gazebo>
     <link name="lobase">
         <visual>
@@ -60,7 +57,4 @@
         </xacro:inertial_box>
     </link>
-    <gazebo reference="lobase">
-      <material>Gazebo/white</material>
-    </gazebo>
     <link name="lidar">
         <visual>
@@ -80,7 +74,4 @@
         </xacro:inertial_cylinder>
     </link>
-    <gazebo reference="lidar">
-      <material>Gazebo/blue</material>
-    </gazebo>
     <link name="pipe">
         <visual>
@@ -101,7 +92,4 @@
         </xacro:inertial_box>
     </link>
-    <gazebo reference="pipe">
-      <material>Gazebo/orange</material>
-    </gazebo>
     <link name="front_left">
       <visual>
@@ -121,7 +109,4 @@
         </xacro:inertial_cylinder>
     </link>
-    <gazebo reference="front_left">
-      <material>Gazebo/black</material>
-    </gazebo>
     <link name="front_right">
       <visual>
@@ -141,7 +126,4 @@
         </xacro:inertial_cylinder>
     </link>
-    <gazebo reference="front_right">
-      <material>Gazebo/black</material>
-    </gazebo>
     <link name="rear_right">
       <visual>
@@ -161,7 +143,4 @@
         </xacro:inertial_cylinder>
     </link>
-    <gazebo reference="rear_right">
-      <material>Gazebo/black</material>
-    </gazebo>
     <link name="rear_left">
       <visual>
@@ -181,7 +160,4 @@
         </xacro:inertial_cylinder>
     </link>
-    <gazebo reference="rear_left">
-      <material>Gazebo/black</material>
-    </gazebo>
     <joint name="base_joint" type="fixed">
        <parent link="base_footprint"/>
@@ -228,3 +204,27 @@
        <origin xyz="0.1 0.25 0.625" rpy="0 0 0" />
     </joint>
+    <gazebo reference="lidar">
+        <material>Gazebo/Blue</material>
+    </gazebo>
+    <gazebo reference="base_link">
+          <material>Gazebo/Green</material>
+    </gazebo>
+    <gazebo reference="lobase">
+      <material>Gazebo/white</material>
+    </gazebo>
+    <gazebo reference="pipe">
+      <material>Gazebo/Orange</material>
+    </gazebo>
+    <gazebo reference="front_left">
+      <material>Gazebo/Black</material>
+    </gazebo>
+    <gazebo reference="front_right">
+      <material>Gazebo/Black</material>
+    </gazebo>
+    <gazebo reference="rear_left">
+      <material>Gazebo/Black</material>
+    </gazebo>
+    <gazebo reference="rear_right">
+      <material>Gazebo/Black</material>
+    </gazebo>
 </robot>

Commit message: created core URDF

File: description/robot_core.xacro (robot description, xacro)
@@ -11,4 +11,7 @@
         <color rgba="1 1 1 1" />
     </material>
+    <material name="red">
+        <color rgba="1 0.2 0.2 0.2" />
+    </material>
     <material name="orange">
         <color rgba="1 0.3 0.1 1"/>
@@ -211,5 +214,5 @@
     </gazebo>
     <gazebo reference="lobase">
-      <material>Gazebo/white</material>
+      <material>Gazebo/Red</material>
     </gazebo>
     <gazebo reference="pipe">

Commit message: created core URDF

File: description/robot_core.xacro (robot description, xacro)
@@ -170,5 +170,5 @@
     <joint name="base_front_left_wheel_joint" type="continuous">
       <parent link="base_link"/>
-      <child link="front_left"/>
+      <child link="front_left_wheel"/>
       <origin xyz="0.18 0.06 -0.175" rpy="0 0 0"/>
       <axis xyz="0 1 0"/>
@@ -176,5 +176,5 @@
     <joint name="base_front_right_wheel_joint" type="continuous">
       <parent link="base_link"/>
-      <child link="front_right"/>
+      <child link="front_right_wheel"/>
       <origin xyz="0.18 0.44 -0.175" rpy="0 0 0"/>
       <axis xyz="0 1 0"/>
@@ -182,5 +182,5 @@
     <joint name="base_rear_right_wheel_joint" type="continuous">
       <parent link="base_link"/>
-      <child link="rear_right"/>
+      <child link="rear_right_wheel"/>
       <origin xyz="0.57 0.44 -0.175" rpy="0 0 0"/>
       <axis xyz="0 1 0"/>
@@ -188,5 +188,5 @@
     <joint name="base_rear_left_wheel_joint" type="continuous">
       <parent link="base_link"/>
-      <child link="rear_left"/>
+      <child link="rear_left_wheel"/>
       <origin xyz="0.57 0.06 -0.175" rpy="0 0 0"/>
       <axis xyz="0 1 0"/>

Commit message: created core URDF

File: description/robot_core.xacro (robot description, xacro)
@@ -166,10 +166,10 @@
        <parent link="base_footprint"/>
        <child link="base_link"/>
-       <origin xyz="-0.375 -0.25 0.327" rpy="0 0 0" />
+       <origin xyz="-0.375 -0.25 0.3" rpy="0 0 0" />
     </joint>
     <joint name="base_front_left_wheel_joint" type="continuous">
       <parent link="base_link"/>
       <child link="front_left_wheel"/>
-      <origin xyz="0.18 0.06 -0.175" rpy="0 0 0"/>
+      <origin xyz="0.18 0.06 -0.15" rpy="0 0 0"/>
       <axis xyz="0 1 0"/>
     </joint>
@@ -177,5 +177,5 @@
       <parent link="base_link"/>
       <child link="front_right_wheel"/>
-      <origin xyz="0.18 0.44 -0.175" rpy="0 0 0"/>
+      <origin xyz="0.18 0.44 -0.15" rpy="0 0 0"/>
       <axis xyz="0 1 0"/>
     </joint>
@@ -183,5 +183,5 @@
       <parent link="base_link"/>
       <child link="rear_right_wheel"/>
-      <origin xyz="0.57 0.44 -0.175" rpy="0 0 0"/>
+      <origin xyz="0.57 0.44 -0.15" rpy="0 0 0"/>
       <axis xyz="0 1 0"/>
     </joint>
@@ -189,5 +189,5 @@
       <parent link="base_link"/>
       <child link="rear_left_wheel"/>
-      <origin xyz="0.57 0.06 -0.175" rpy="0 0 0"/>
+      <origin xyz="0.57 0.06 -0.15" rpy="0 0 0"/>
       <axis xyz="0 1 0"/>
     </joint>
@@ -195,5 +195,5 @@
        <parent link="base_link"/>
        <child link="lobase"/>
-       <origin xyz="0.375 0.25 -0.1" rpy="0 0 0"/>
+       <origin xyz="0.375 0.25 -0.075" rpy="0 0 0"/>
     </joint>
     <joint name="base_lidar_joint" type="fixed">

Commit message: created core URDF

File: description/robot_core.xacro (robot description, xacro)
@@ -109,5 +109,5 @@
         </collision>
         <xacro:inertial_cylinder mass="0.3" length="0.08" radius="0.15">
-            <origin xyz="0 0 -.04" rpy="0 0 0"/>
+            <origin xyz="0 0 0" rpy="0 0 0"/>
         </xacro:inertial_cylinder>
     </link>
@@ -126,5 +126,5 @@
         </collision>
         <xacro:inertial_cylinder mass="0.3" length="0.08" radius="0.15">
-            <origin xyz="0 0 -.04" rpy="0 0 0"/>
+            <origin xyz="0 0 0" rpy="0 0 0"/>
         </xacro:inertial_cylinder>
     </link>
@@ -143,5 +143,5 @@
         </collision>
         <xacro:inertial_cylinder mass="0.3" length="0.08" radius="0.15">
-            <origin xyz="0 0 -.04" rpy="0 0 0"/>
+            <origin xyz="0 0 0" rpy="0 0 0"/>
         </xacro:inertial_cylinder>
     </link>
@@ -160,5 +160,5 @@
         </collision>
         <xacro:inertial_cylinder mass="0.3" length="0.08" radius="0.15">
-            <origin xyz="0 0 -.04" rpy="0 0 0"/>
+            <origin xyz="0 0 0" rpy="0 0 0"/>
         </xacro:inertial_cylinder>
     </link>

Commit message: created core URDF

File: description/robot_core.xacro (robot description, xacro)
@@ -144,5 +144,5 @@
     </link>
     <!-- FRONT LEFT WHEEL LINK -->
-    <joint name="front_left_wheel_joint" type="continuous">
+    <joint name="front_left_wheel_joint" type="fixed">
         <parent link="base_link"/>
         <child link="front_left_wheel"/>
@@ -190,5 +190,5 @@
     </link>
     <!-- FRONT RIGHT WHEEL LINK -->
-    <joint name="front_right_wheel_joint" type="continuous">
+    <joint name="front_right_wheel_joint" type="fixed">
         <parent link="base_link"/>
         <child link="front_right_wheel"/>

Commit message: created core URDF

File: description/robot_core.xacro (robot description, xacro)
@@ -98,26 +98,4 @@
         </xacro:inertial_box>
     </link>
-    <!-- LIDAR LINK -->
-    <joint name="lidar_joint" type="fixed">
-        <parent link="base_link"/>
-        <child link="lidar"/>
-        <origin xyz="0.275 0 0.465"  />
-    </joint>
-    <link name="lidar">
-        <visual>
-            <geometry>
-                <cylinder radius="0.05" length="0.03"/>
-            </geometry>
-            <material name="blue"/>
-        </visual>
-        <collision>
-            <geometry>
-                <cylinder radius="0.05" length="0.03"/>
-            </geometry>
-        </collision>
-        <xacro:inertial_cylinder mass="0.1" length="0.03" radius="0.05">
-            <origin xyz="0 0 0" rpy="0 0 0"/>
-        </xacro:inertial_cylinder>
-    </link>
     <!-- REAR LEFT WHEEL LINK -->
     <joint name="rear_left_wheel_joint" type="continuous">
@@ -212,7 +190,4 @@
         </xacro:inertial_cylinder>
     </link>
-    <gazebo reference="lidar">
-        <material>Gazebo/Blue</material>
-    </gazebo>
     <gazebo reference="chassis">
           <material>Gazebo/White</material>
