Commit message: created core URDF

File: description/gazebo_control.xacro (robot description, xacro)
@@ -1,22 +1,21 @@
 <?xml version="1.0"?>
-<robot xmlns:xacro="http://www.ros.org/wiki/xacro"  >
-<gazebo>
-    <plugin name="diff_drive" filename="libgazebo_ros_diff_drive.so">
-         <!--wheel info-->
-         <front_left_joint>front_left_joint</front_left_joint>
-         <rear_left_joint>rear_left_joint</raer_left_joint>
-         <front_right_joint>front_right_joint</front_right_joint>
-         <raer_right_joint>rear_right_joint</rear_right_joint>
-         <wheel_separation>0.3</wheel_separation>
-         <wheel_diameter>0.3</wheel_diameter>
-         <!-- Limits -->
+<robot xmlns:xacro="http://www.ros.org/wiki/xacro">
+    <gazebo>
+        <plugin name="diff_drive" filename="libgazebo_ros_diff_drive.so">
+            <!-- Wheel Information -->
+            <left_joint>left_wheel_joint</left_joint>
+            <right_joint>right_wheel_joint</right_joint>
+            <wheel_separation>0.3</wheel_separation>
+            <wheel_diameter>0.3</wheel_diameter>
+            <!-- Limits -->
             <max_wheel_torque>200</max_wheel_torque>
             <max_wheel_acceleration>10.0</max_wheel_acceleration>
             <!-- Output -->
             <odometry_frame>odom</odometry_frame>
-            <robot_base_frame>base_footprint_link</robot_base_frame>
+            <robot_base_frame>base_link</robot_base_frame>
             <publish_odom>true</publish_odom>
             <publish_odom_tf>true</publish_odom_tf>
             <publish_wheel_tf>true</publish_wheel_tf>
-    </plugin>
+        </plugin>
+    </gazebo>
 </robot>

File: description/robot_core.xacro (robot description, xacro)
@@ -95,56 +95,56 @@
         </xacro:inertial_box>
     </link>
-    <link name="front_left">
-      <visual>
-         <geometry>
-             <cylinder radius="0.15" length="0.08"/>
-         </geometry>
-         <origin xyz="0 0 0" rpy="1.57 0 0"/>
-         <material name="black"/>
-      </visual>
-      <collision>
-            <geometry>
-                <cylinder radius="0.15" length="0.08"/>
-            </geometry>
-        </collision>
-        <xacro:inertial_cylinder mass="0.3" length="0.08" radius="0.15">
-            <origin xyz="0 0 0" rpy="0 0 0"/>
-        </xacro:inertial_cylinder>
-    </link>
-    <link name="front_right">
-      <visual>
-         <geometry>
-             <cylinder radius="0.15" length="0.08"/>
-         </geometry>
-         <origin xyz="0 0 0" rpy="1.57 0 0"/>
-         <material name="black"/>
-      </visual>
-      <collision>
-            <geometry>
-                <cylinder radius="0.15" length="0.08"/>
-            </geometry>
-        </collision>
-        <xacro:inertial_cylinder mass="0.3" length="0.08" radius="0.15">
-            <origin xyz="0 0 0" rpy="0 0 0"/>
-        </xacro:inertial_cylinder>
-    </link>
-    <link name="rear_right">
-      <visual>
-         <geometry>
-             <cylinder radius="0.15" length="0.08"/>
-         </geometry>
-         <origin xyz="0 0 0" rpy="1.57 0 0"/>
-         <material name="black"/>
-      </visual>
-      <collision>
-            <geometry>
-                <cylinder radius="0.15" length="0.08"/>
-            </geometry>
-        </collision>
-        <xacro:inertial_cylinder mass="0.3" length="0.08" radius="0.15">
-            <origin xyz="0 0 0" rpy="0 0 0"/>
-        </xacro:inertial_cylinder>
-    </link>
-    <link name="rear_left">
+    <link name="front_left_wheel">
+      <visual>
+         <geometry>
+             <cylinder radius="0.15" length="0.08"/>
+         </geometry>
+         <origin xyz="0 0 0" rpy="1.57 0 0"/>
+         <material name="black"/>
+      </visual>
+      <collision>
+            <geometry>
+                <cylinder radius="0.15" length="0.08"/>
+            </geometry>
+        </collision>
+        <xacro:inertial_cylinder mass="0.3" length="0.08" radius="0.15">
+            <origin xyz="0 0 0" rpy="0 0 0"/>
+        </xacro:inertial_cylinder>
+    </link>
+    <link name="front_right_wheel">
+      <visual>
+         <geometry>
+             <cylinder radius="0.15" length="0.08"/>
+         </geometry>
+         <origin xyz="0 0 0" rpy="1.57 0 0"/>
+         <material name="black"/>
+      </visual>
+      <collision>
+            <geometry>
+                <cylinder radius="0.15" length="0.08"/>
+            </geometry>
+        </collision>
+        <xacro:inertial_cylinder mass="0.3" length="0.08" radius="0.15">
+            <origin xyz="0 0 0" rpy="0 0 0"/>
+        </xacro:inertial_cylinder>
+    </link>
+    <link name="rear_right_wheel">
+      <visual>
+         <geometry>
+             <cylinder radius="0.15" length="0.08"/>
+         </geometry>
+         <origin xyz="0 0 0" rpy="1.57 0 0"/>
+         <material name="black"/>
+      </visual>
+      <collision>
+            <geometry>
+                <cylinder radius="0.15" length="0.08"/>
+            </geometry>
+        </collision>
+        <xacro:inertial_cylinder mass="0.3" length="0.08" radius="0.15">
+            <origin xyz="0 0 0" rpy="0 0 0"/>
+        </xacro:inertial_cylinder>
+    </link>
+    <link name="rear_left_wheel">
       <visual>
          <geometry>
@@ -168,5 +168,5 @@
        <origin xyz="-0.375 -0.25 0.327" rpy="0 0 0" />
     </joint>
-    <joint name="base_front_left_joint" type="continuous">
+    <joint name="base_front_left_wheel_joint" type="continuous">
       <parent link="base_link"/>
       <child link="front_left"/>
@@ -174,5 +174,5 @@
       <axis xyz="0 1 0"/>
     </joint>
-    <joint name="base_front_right_joint" type="continuous">
+    <joint name="base_front_right_wheel_joint" type="continuous">
       <parent link="base_link"/>
       <child link="front_right"/>
@@ -180,5 +180,5 @@
       <axis xyz="0 1 0"/>
     </joint>
-    <joint name="base_rear_right_joint" type="continuous">
+    <joint name="base_rear_right_wheel_joint" type="continuous">
       <parent link="base_link"/>
       <child link="rear_right"/>
@@ -186,5 +186,5 @@
       <axis xyz="0 1 0"/>
     </joint>
-    <joint name="base_rear_left_joint" type="continuous">
+    <joint name="base_rear_left_wheel_joint" type="continuous">
       <parent link="base_link"/>
       <child link="rear_left"/>
@@ -219,14 +219,14 @@
       <material>Gazebo/Orange</material>
     </gazebo>
-    <gazebo reference="front_left">
-      <material>Gazebo/Black</material>
-    </gazebo>
-    <gazebo reference="front_right">
-      <material>Gazebo/Black</material>
-    </gazebo>
-    <gazebo reference="rear_left">
-      <material>Gazebo/Black</material>
-    </gazebo>
-    <gazebo reference="rear_right">
+    <gazebo reference="front_left_wheel">
+      <material>Gazebo/Black</material>
+    </gazebo>
+    <gazebo reference="front_right_wheel">
+      <material>Gazebo/Black</material>
+    </gazebo>
+    <gazebo reference="rear_left_wheel">
+      <material>Gazebo/Black</material>
+    </gazebo>
+    <gazebo reference="rear_right_wheel">
       <material>Gazebo/Black</material>
     </gazebo>

Commit message: created core URDF

File: description/gazebo_control.xacro (robot description, xacro)
@@ -4,6 +4,6 @@
         <plugin name="diff_drive" filename="libgazebo_ros_diff_drive.so">
             <!-- Wheel Information -->
-            <left_joint>left_wheel_joint</left_joint>
-            <right_joint>right_wheel_joint</right_joint>
+            <left_joint>base_rear_left_wheel_joint</left_joint>
+            <right_joint>base_rear_right_wheel_joint</right_joint>
             <wheel_separation>0.3</wheel_separation>
             <wheel_diameter>0.3</wheel_diameter>

File: description/robot_core.xacro (robot description, xacro)
@@ -109,5 +109,5 @@
         </collision>
         <xacro:inertial_cylinder mass="0.3" length="0.08" radius="0.15">
-            <origin xyz="0 0 0" rpy="0 0 0"/>
+            <origin xyz="0 0 -.04" rpy="0 0 0"/>
         </xacro:inertial_cylinder>
     </link>
@@ -126,5 +126,5 @@
         </collision>
         <xacro:inertial_cylinder mass="0.3" length="0.08" radius="0.15">
-            <origin xyz="0 0 0" rpy="0 0 0"/>
+            <origin xyz="0 0 -.04" rpy="0 0 0"/>
         </xacro:inertial_cylinder>
     </link>
@@ -143,5 +143,5 @@
         </collision>
         <xacro:inertial_cylinder mass="0.3" length="0.08" radius="0.15">
-            <origin xyz="0 0 0" rpy="0 0 0"/>
+            <origin xyz="0 0 -.04" rpy="0 0 0"/>
         </xacro:inertial_cylinder>
     </link>
@@ -160,5 +160,5 @@
         </collision>
         <xacro:inertial_cylinder mass="0.3" length="0.08" radius="0.15">
-            <origin xyz="0 0 0" rpy="0 0 0"/>
+            <origin xyz="0 0 -.04" rpy="0 0 0"/>
         </xacro:inertial_cylinder>
     </link>
@@ -221,13 +221,21 @@
     <gazebo reference="front_left_wheel">
       <material>Gazebo/Black</material>
+      <mu1 value="0.001"/>
+      <mu2 value="0.001"/>
     </gazebo>
     <gazebo reference="front_right_wheel">
       <material>Gazebo/Black</material>
+      <mu1 value="0.001"/>
+      <mu2 value="0.001"/>
     </gazebo>
     <gazebo reference="rear_left_wheel">
       <material>Gazebo/Black</material>
+      <mu1 value="0.001"/>
+      <mu2 value="0.001"/>
     </gazebo>
     <gazebo reference="rear_right_wheel">
       <material>Gazebo/Black</material>
+      <mu1 value="0.001"/>
+      <mu2 value="0.001"/>
     </gazebo>
 </robot>

Commit message: created core UDRF

File: description/gazebo_control.xacro (robot description, xacro)
@@ -4,6 +4,6 @@
         <plugin name="diff_drive" filename="libgazebo_ros_diff_drive.so">
             <!-- Wheel Information -->
-            <left_joint>base_rear_left_wheel_joint</left_joint>
-            <right_joint>base_rear_right_wheel_joint</right_joint>
+            <left_joint>rear_left_wheel_joint</left_joint>
+            <right_joint>rear_right_wheel_joint</right_joint>
             <wheel_separation>0.3</wheel_separation>
             <wheel_diameter>0.3</wheel_diameter>
@@ -13,5 +13,5 @@
             <!-- Output -->
             <odometry_frame>odom</odometry_frame>
-            <robot_base_frame>base_footprint_link</robot_base_frame>
+            <robot_base_frame>base_link</robot_base_frame>
             <publish_odom>true</publish_odom>
             <publish_odom_tf>true</publish_odom_tf>

File: description/robot_core.xacro (robot description, xacro)
@@ -23,53 +23,96 @@
         <color rgba="0 0 0 1"/>
     </material>
-    <link name="base_footprint" />
+    <!-- BASE LINK -->
     <link name="base_link">
-        <visual>
-            <geometry>
-                <box size="0.75 0.5 0.3" />
-            </geometry>
-            <origin xyz="0.375 0.25 0.15" rpy="0 0 0" />
-             <material name="green" />
-        </visual>
-        <collision>
-            <origin xyz="0.375 0.25 0.15"/>
+    </link>
+    <!-- CHASSIS LINK -->
+    <joint name="chassis_joint" type="fixed">
+        <parent link="base_link"/>
+        <child link="chassis"/>
+        <origin xyz="0 0 0.3"/>
+    </joint>
+    <link name="chassis">
+        <visual>
+            <origin xyz="0 0 0"/>
             <geometry>
                 <box size="0.75 0.5 0.3"/>
             </geometry>
+            <material name="white"/>
+        </visual>
+        <collision>
+            <origin xyz="0 0 0"/>
+            <geometry>
+                <box size="0.75 0.5 0.3"/>
+            </geometry>
         </collision>
         <xacro:inertial_box mass="0.5" x="0.75" y="0.5" z="0.3">
-            <origin xyz="0.375 0.25 0.15" rpy="0 0 0"/>
+            <origin xyz="0 0 0" rpy="0 0 0"/>
         </xacro:inertial_box>
     </link>
-    <link name="lobase">
-        <visual>
-            <geometry>
-                <box size="0.6 0.3 0.15" />
-            </geometry>
-            <origin xyz="0 0 0" rpy="0 0 0" />
-            <material name="red" />
-        </visual>
-        <collision>
+    <!-- SUB_CHASSIS LINK -->
+    <joint name="sub_chassis_joint" type="fixed">
+        <parent link="base_link"/>
+        <child link="sub_chassis"/>
+        <origin xyz="0 0 0.075"/>
+    </joint>
+    <link name="sub_chassis">
+        <visual>
             <origin xyz="0 0 0"/>
             <geometry>
                 <box size="0.6 0.3 0.15"/>
             </geometry>
-        </collision>
-        <xacro:inertial_box mass="0.5" x="0.6" y="0.3" z="0.15">
+            <material name="grey"/>
+        </visual>
+        <collision>
+            <origin xyz="0 0 0"/>
+            <geometry>
+                <box size="0.6 0.3 0.15"/>
+            </geometry>
+        </collision>
+        <xacro:inertial_box mass="0.35" x="0.6" y="0.3" z="0.15">
             <origin xyz="0 0 0" rpy="0 0 0"/>
         </xacro:inertial_box>
     </link>
+    <!-- PIPE LINK -->
+    <joint name="pipe_joint" type="fixed">
+        <parent link="base_link"/>
+        <child link="pipe"/>
+        <origin xyz="-0.275 0 0.775"/>
+    </joint>
+    <link name="pipe">
+        <visual>
+            <origin xyz="0 0 0"/>
+            <geometry>
+                <box size="0.04 0.04 0.65"/>
+            </geometry>
+            <material name="orange"/>
+        </visual>
+        <collision>
+            <origin xyz="0 0 0"/>
+            <geometry>
+                <box size="0.04 0.04 .65"/>
+            </geometry>
+        </collision>
+        <xacro:inertial_box mass="0.2" x="0.04" y="0.04" z="0.65">
+            <origin xyz="0 0 0" rpy="0 0 0"/>
+        </xacro:inertial_box>
+    </link>
+    <!-- LIDAR LINK -->
+    <joint name="lidar_joint" type="fixed">
+        <parent link="base_link"/>
+        <child link="lidar"/>
+        <origin xyz="0.275 0 0.465"  />
+    </joint>
     <link name="lidar">
         <visual>
             <geometry>
-                <cylinder radius="0.05" length="0.03" />
-            </geometry>
-            <origin xyz="0 0 0" rpy="0 0 0" />
-            <material name="blue" />
-        </visual>
-        <collision>
-            <geometry>
                 <cylinder radius="0.05" length="0.03"/>
             </geometry>
+            <material name="blue"/>
+        </visual>
+        <collision>
+            <geometry>
+                <cylinder radius="0.05" length="0.03"/>
+            </geometry>
         </collision>
         <xacro:inertial_cylinder mass="0.1" length="0.03" radius="0.05">
@@ -77,142 +120,104 @@
         </xacro:inertial_cylinder>
     </link>
-    <link name="pipe">
-        <visual>
-            <geometry>
-              <box size="0.04 0.04 .65"/>
-            </geometry>
-            <origin xyz="0 0 0" rpy="0 0 0"/>
-            <material name="orange"/>
-        </visual>
-        <collision>
-            <origin xyz="0 0 0"/>
-            <geometry>
-                <box size="0.04 0.04 0.65"/>
-            </geometry>
-        </collision>
-        <xacro:inertial_box mass="0.25" x="0.04" y="0.04" z="0.65">
-            <origin xyz="0 0 0" rpy="0 0 0"/>
-        </xacro:inertial_box>
-    </link>
+    <!-- REAR LEFT WHEEL LINK -->
+    <joint name="rear_left_wheel_joint" type="continuous">
+        <parent link="base_link"/>
+        <child link="rear_left_wheel"/>
+        <origin xyz="0.2 -0.19 0" rpy="-${pi/2} 0 0" />
+        <axis xyz="0 0 -1"/>
+    </joint>
+    <link name="rear_left_wheel">
+        <visual>
+            <geometry>
+                <cylinder radius="0.14" length="0.08"/>
+            </geometry>
+            <material name="black"/>
+        </visual>
+        <collision>
+            <geometry>
+                <cylinder radius="0.14" length="0.08"/>
+            </geometry>
+        </collision>
+        <xacro:inertial_cylinder mass="0.1" length="0.08" radius="0.14">
+            <origin xyz="0 0 0" rpy="0 0 0"/>
+        </xacro:inertial_cylinder>
+    </link>
+    <!-- FRONT LEFT WHEEL LINK -->
+    <joint name="front_left_wheel_joint" type="continuous">
+        <parent link="base_link"/>
+        <child link="front_left_wheel"/>
+        <origin xyz="-0.2 -0.19 0" rpy="-${pi/2} 0 0" />
+        <axis xyz="0 0 -1"/>
+    </joint>
     <link name="front_left_wheel">
-      <visual>
-         <geometry>
-             <cylinder radius="0.15" length="0.08"/>
-         </geometry>
-         <origin xyz="0 0 0" rpy="1.57 0 0"/>
-         <material name="black"/>
-      </visual>
-      <collision>
-            <geometry>
-                <cylinder radius="0.15" length="0.08"/>
-            </geometry>
-        </collision>
-        <xacro:inertial_cylinder mass="0.3" length="0.08" radius="0.15">
-            <origin xyz="0 0 0" rpy="0 0 0"/>
-        </xacro:inertial_cylinder>
-    </link>
+        <visual>
+            <geometry>
+                <cylinder radius="0.14" length="0.08"/>
+            </geometry>
+            <material name="black"/>
+        </visual>
+        <collision>
+            <geometry>
+                <cylinder radius="0.14" length="0.08"/>
+            </geometry>
+        </collision>
+        <xacro:inertial_cylinder mass="0.1" length="0.08" radius="0.14">
+            <origin xyz="0 0 0" rpy="0 0 0"/>
+        </xacro:inertial_cylinder>
+    </link>
+    <!-- REAR RIGHT WHEEL LINK -->
+    <joint name="rear_right_wheel_joint" type="continuous">
+        <parent link="base_link"/>
+        <child link="rear_right_wheel"/>
+        <origin xyz="0.2 0.19 0" rpy="${pi/2} 0 0" />
+        <axis xyz="0 0 1"/>
+    </joint>
+    <link name="rear_right_wheel">
+        <visual>
+            <geometry>
+                <cylinder radius="0.14" length="0.08"/>
+            </geometry>
+            <material name="black"/>
+        </visual>
+        <collision>
+            <geometry>
+                <cylinder radius="0.14" length="0.08"/>
+            </geometry>
+        </collision>
+        <xacro:inertial_cylinder mass="0.1" length="0.08" radius="0.14">
+            <origin xyz="0 0 0" rpy="0 0 0"/>
+        </xacro:inertial_cylinder>
+    </link>
+    <!-- FRONT RIGHT WHEEL LINK -->
+    <joint name="front_right_wheel_joint" type="continuous">
+        <parent link="base_link"/>
+        <child link="front_right_wheel"/>
+        <origin xyz="-0.2 0.19 0" rpy="${pi/2} 0 0" />
+        <axis xyz="0 0 1"/>
+    </joint>
     <link name="front_right_wheel">
-      <visual>
-         <geometry>
-             <cylinder radius="0.15" length="0.08"/>
-         </geometry>
-         <origin xyz="0 0 0" rpy="1.57 0 0"/>
-         <material name="black"/>
-      </visual>
-      <collision>
-            <geometry>
-                <cylinder radius="0.15" length="0.08"/>
-            </geometry>
-        </collision>
-        <xacro:inertial_cylinder mass="0.3" length="0.08" radius="0.15">
-            <origin xyz="0 0 0" rpy="0 0 0"/>
-        </xacro:inertial_cylinder>
-    </link>
-    <link name="rear_right_wheel">
-      <visual>
-         <geometry>
-             <cylinder radius="0.15" length="0.08"/>
-         </geometry>
-         <origin xyz="0 0 0" rpy="1.57 0 0"/>
-         <material name="black"/>
-      </visual>
-      <collision>
-            <geometry>
-                <cylinder radius="0.15" length="0.08"/>
-            </geometry>
-        </collision>
-        <xacro:inertial_cylinder mass="0.3" length="0.08" radius="0.15">
-            <origin xyz="0 0 0" rpy="0 0 0"/>
-        </xacro:inertial_cylinder>
-    </link>
-    <link name="rear_left_wheel">
-      <visual>
-         <geometry>
-             <cylinder radius="0.15" length="0.08"/>
-         </geometry>
-         <origin xyz="0 0 0" rpy="1.57 0 0"/>
-         <material name="black"/>
-      </visual>
-      <collision>
-            <geometry>
-                <cylinder radius="0.15" length="0.08"/>
-            </geometry>
-        </collision>
-        <xacro:inertial_cylinder mass="0.3" length="0.08" radius="0.15">
-            <origin xyz="0 0 0" rpy="0 0 0"/>
-        </xacro:inertial_cylinder>
-    </link>
-    <joint name="base_joint" type="fixed">
-       <parent link="base_footprint"/>
-       <child link="base_link"/>
-       <origin xyz="-0.375 -0.25 0.3" rpy="0 0 0" />
-    </joint>
-    <joint name="base_front_left_wheel_joint" type="continuous">
-      <parent link="base_link"/>
-      <child link="front_left_wheel"/>
-      <origin xyz="0.18 0.06 -0.15" rpy="0 0 0"/>
-      <axis xyz="0 1 0"/>
-    </joint>
-    <joint name="base_front_right_wheel_joint" type="continuous">
-      <parent link="base_link"/>
-      <child link="front_right_wheel"/>
-      <origin xyz="0.18 0.44 -0.15" rpy="0 0 0"/>
-      <axis xyz="0 1 0"/>
-    </joint>
-    <joint name="base_rear_right_wheel_joint" type="continuous">
-      <parent link="base_link"/>
-      <child link="rear_right_wheel"/>
-      <origin xyz="0.57 0.44 -0.15" rpy="0 0 0"/>
-      <axis xyz="0 1 0"/>
-    </joint>
-    <joint name="base_rear_left_wheel_joint" type="continuous">
-      <parent link="base_link"/>
-      <child link="rear_left_wheel"/>
-      <origin xyz="0.57 0.06 -0.15" rpy="0 0 0"/>
-      <axis xyz="0 1 0"/>
-    </joint>
-    <joint name="base_lobase_joint" type="fixed">
-       <parent link="base_link"/>
-       <child link="lobase"/>
-       <origin xyz="0.375 0.25 -0.075" rpy="0 0 0"/>
-    </joint>
-    <joint name="base_lidar_joint" type="fixed">
-       <parent link="base_link"/>
-       <child link="lidar"/>
-       <origin xyz="0.65 0.25 0.315" rpy="0 0 0"/>
-    </joint>
-    <joint name="base_pipe_joint" type="fixed">
-       <parent link="base_link"/>
-       <child link="pipe"/>
-       <origin xyz="0.1 0.25 0.625" rpy="0 0 0" />
-    </joint>
+        <visual>
+            <geometry>
+                <cylinder radius="0.14" length="0.08"/>
+            </geometry>
+            <material name="black"/>
+        </visual>
+        <collision>
+            <geometry>
+                <cylinder radius="0.14" length="0.08"/>
+            </geometry>
+        </collision>
+        <xacro:inertial_cylinder mass="0.1" length="0.08" radius="0.14">
+            <origin xyz="0 0 0" rpy="0 0 0"/>
+        </xacro:inertial_cylinder>
+    </link>
     <gazebo reference="lidar">
         <material>Gazebo/Blue</material>
     </gazebo>
-    <gazebo reference="base_link">
-          <material>Gazebo/Green</material>
-    </gazebo>
-    <gazebo reference="lobase">
-      <material>Gazebo/Red</material>
+    <gazebo reference="chassis">
+          <material>Gazebo/White</material>
+    </gazebo>
+    <gazebo reference="sub_chassis">
+      <material>Gazebo/Grey</material>
     </gazebo>
     <gazebo reference="pipe">
@@ -231,11 +236,7 @@
     <gazebo reference="rear_left_wheel">
       <material>Gazebo/Black</material>
-      <mu1 value="0.001"/>
-      <mu2 value="0.001"/>
     </gazebo>
     <gazebo reference="rear_right_wheel">
       <material>Gazebo/Black</material>
-      <mu1 value="0.001"/>
-      <mu2 value="0.001"/>
     </gazebo>
 </robot>
