Commit message: created core urdf

File: description/gazebo_control.xacro (robot description, xacro)
@@ -4,6 +4,6 @@
         <plugin name="diff_drive" filename="libgazebo_ros_diff_drive.so">
             <!-- Wheel Information -->
-            <left_joint>rear_left_wheel_joint</left_joint>
-            <right_joint>rear_right_wheel_joint</right_joint>
+            <left_joint>front_left_wheel_joint</left_joint>
+            <right_joint>front_right_wheel_joint</right_joint>
             <wheel_separation>0.38</wheel_separation>
             <wheel_diameter>0.28</wheel_diameter>

File: description/robot.urdf.xacro (robot description, xacro)
@@ -4,3 +4,4 @@
     <xacro:include filename="gazebo_control.xacro" />
     <xacro:include filename="lidar.xacro" />
+    <xacro:include filename="camera.xacro" />
 </robot>

File: description/robot_core.xacro (robot description, xacro)
@@ -98,9 +98,32 @@
         </xacro:inertial_box>
     </link>
+    <!-- FRONT RIGHT WHEEL LINK -->
+    <joint name="front_right_wheel_joint" type="continuous">
+        <parent link="base_link"/>
+        <child link="front_right_wheel"/>
+        <origin xyz="0.2 -0.19 0" rpy="${pi/2} 0 0" />
+        <axis xyz="0 0 -1"/>
+    </joint>
+    <link name="front_right_wheel">
+        <visual>
+            <geometry>
+                <cylinder radius="0.14" length="0.08"/>
+            </geometry>
+            <material name="black"/>
+        </visual>
+        <collision>
+            <geometry>
+                <cylinder radius="0.14" length="0.08"/>
+            </geometry>
+        </collision>
+        <xacro:inertial_cylinder mass="0.1" length="0.08" radius="0.14">
+            <origin xyz="0 0 0" rpy="0 0 0"/>
+        </xacro:inertial_cylinder>
+    </link>
     <!-- REAR LEFT WHEEL LINK -->
-    <joint name="rear_left_wheel_joint" type="continuous">
+    <joint name="rear_left_wheel_joint" type="fixed">
         <parent link="base_link"/>
         <child link="rear_left_wheel"/>
-        <origin xyz="0.2 -0.19 0" rpy="-${pi/2} 0 0" />
+        <origin xyz="-0.2 -0.19 0" rpy="${pi/2} 0 0" />
         <axis xyz="0 0 -1"/>
     </joint>
@@ -122,9 +145,9 @@
     </link>
     <!-- FRONT LEFT WHEEL LINK -->
-    <joint name="front_left_wheel_joint" type="fixed">
+    <joint name="front_left_wheel_joint" type="continuous">
         <parent link="base_link"/>
         <child link="front_left_wheel"/>
-        <origin xyz="-0.2 -0.19 0" rpy="-${pi/2} 0 0" />
-        <axis xyz="0 0 -1"/>
+        <origin xyz="0.2 0.19 0" rpy="-${pi/2} 0 0" />
+        <axis xyz="0 0 1"/>
     </joint>
     <link name="front_left_wheel">
@@ -145,34 +168,11 @@
     </link>
     <!-- REAR RIGHT WHEEL LINK -->
-    <joint name="rear_right_wheel_joint" type="continuous">
+    <joint name="rear_right_wheel_joint" type="fixed">
         <parent link="base_link"/>
         <child link="rear_right_wheel"/>
-        <origin xyz="0.2 0.19 0" rpy="${pi/2} 0 0" />
+        <origin xyz="-0.2 0.19 0" rpy="-${pi/2} 0 0" />
         <axis xyz="0 0 1"/>
     </joint>
     <link name="rear_right_wheel">
-        <visual>
-            <geometry>
-                <cylinder radius="0.14" length="0.08"/>
-            </geometry>
-            <material name="black"/>
-        </visual>
-        <collision>
-            <geometry>
-                <cylinder radius="0.14" length="0.08"/>
-            </geometry>
-        </collision>
-        <xacro:inertial_cylinder mass="0.1" length="0.08" radius="0.14">
-            <origin xyz="0 0 0" rpy="0 0 0"/>
-        </xacro:inertial_cylinder>
-    </link>
-    <!-- FRONT RIGHT WHEEL LINK -->
-    <joint name="front_right_wheel_joint" type="fixed">
-        <parent link="base_link"/>
-        <child link="front_right_wheel"/>
-        <origin xyz="-0.2 0.19 0" rpy="${pi/2} 0 0" />
-        <axis xyz="0 0 1"/>
-    </joint>
-    <link name="front_right_wheel">
         <visual>
             <geometry>
@@ -199,18 +199,18 @@
       <material>Gazebo/Orange</material>
     </gazebo>
-    <gazebo reference="front_left_wheel">
+    <gazebo reference="rear_left_wheel">
       <material>Gazebo/Black</material>
       <mu1 value="0.001"/>
       <mu2 value="0.001"/>
     </gazebo>
-    <gazebo reference="front_right_wheel">
+    <gazebo reference="rear_right_wheel">
       <material>Gazebo/Black</material>
       <mu1 value="0.001"/>
       <mu2 value="0.001"/>
     </gazebo>
-    <gazebo reference="rear_left_wheel">
-      <material>Gazebo/Black</material>
-    </gazebo>
-    <gazebo reference="rear_right_wheel">
+    <gazebo reference="front_left_wheel">
+      <material>Gazebo/Black</material>
+    </gazebo>
+    <gazebo reference="front_right_wheel">
       <material>Gazebo/Black</material>
     </gazebo>
